Commit message: Added gazebo camera functionality

File: camera_ros2_wrappers/firefly-ros2-wrapper/firefly-ros2-wrapper-description/urdf/firefly_stereo_macro.urdf.xacro (robot description, xacro)
@@ -1,6 +1,8 @@
 <?xml version="1.0"?>
 <robot xmlns:xacro="http://ros.org/wiki/xacro">
+    <!-- Include Gazebo sensor plugins -->
+    <xacro:include filename="$(find firefly-ros2-wrapper-description)/urdf/firefly_stereo_gazebo.urdf.xacro"/>
     <!-- Macro Definition -->
-    <xacro:macro name="firefly_camera">
+    <xacro:macro name="firefly_camera" params="use_gazebo:=true namespace:=firefly">
         <!-- Link: camera body -->
         <link name="firefly_camera_link">
@@ -39,4 +41,8 @@
             <origin xyz="-0.02999871 0.07322070 0.00006055" rpy="${-pi/2} 0 0"/>
         </joint>
+        <!-- Add Gazebo sensor plugins if in simulation -->
+        <xacro:if value="${use_gazebo}">
+            <xacro:firefly_camera_gazebo namespace="${namespace}"/>
+        </xacro:if>
     </xacro:macro>
 </robot>

File: multi_camera_rig_description/urdf/multi_cam_rig_macro.urdf.xacro (robot description, xacro)
@@ -2,5 +2,5 @@
 <robot xmlns:xacro="http://wiki.ros.org/xacro">
     <!-- Macro Definition -->
-    <xacro:macro name="multi_camera_rig">
+    <xacro:macro name="multi_camera_rig" params="use_gazebo:=true">
         <!-- Mounting frame for robot end effector-->
         <link name="multi_camera_rig_mount"/>
@@ -35,5 +35,5 @@
         <!-- Firefly Camera -->
         <xacro:include filename="$(find firefly-ros2-wrapper-description)/urdf/firefly_stereo_macro.urdf.xacro"/>
-        <xacro:firefly_camera/>
+        <xacro:firefly_camera use_gazebo="${use_gazebo}" namespace="firefly"/>
         <joint name="firefly_camera_mount_joint" type="fixed">
             <parent link="multi_camera_rig_link"/>
