Commit message: Implemented gazebo file for firefly camera... currently is functional with the husky xarm mcr package. Will begin fixing up the topics and namespacing for real functionality next. Also updated mesh file paths for proper import and alignment with updated package names for ximea and firefly cameras.

File: camera_ros2_wrappers/firefly-ros2-wrapper/firefly-ros2-wrapper-description/urdf/firefly_stereo_gazebo.urdf.xacro (robot description, xacro)
@@ -3,14 +3,43 @@
     <!-- Gazebo (Ignition) sensor plugins for Firefly stereo camera -->
     <xacro:macro name="firefly_camera_gazebo" params="namespace:=firefly">
+        <!-- Sensors plugin must be loaded by world sdf for vision -->
         <!-- Left Camera Sensor -->
         <gazebo reference="firefly_left_optical_frame">
             <sensor name="firefly_left_camera" type="camera">
+                <update_rate>2</update_rate>
+                <always_on>1</always_on>
+                <visualize>true</visualize>
+                <topic>/camera</topic>
+                <gz_frame_id>firefly_left_optical_frame</gz_frame_id>
+                <!-- <optical_frame_id>firefly_left_optical_frame</optical_frame_id> -->
+                <!-- <camera_info_topic>/firefly_left/camera_info</camera_info_topic> -->
+                <camera>
+                    <horizontal_fov>1.3962634</horizontal_fov>  <!-- 80 degrees -->
+                    <image>
+                        <width>1440</width>
+                        <height>1080</height>
+                        <format>R8G8B8</format>
+                    </image>
+                    <clip>
+                        <near>0.1</near>
+                        <far>300</far>
+                    </clip>
+                    <!-- <noise>
+                        <type>gaussian</type>
+                        <mean>0.0</mean>
+                        <stddev>0.007</stddev>
+                    </noise> -->
+                </camera>
+            </sensor>
+        </gazebo>
+        <!-- Right Camera Sensor -->
+        <!-- <gazebo reference="firefly_right_optical_frame">
+            <sensor name="firefly_right_camera" type="camera">
                 <update_rate>30</update_rate>
                 <always_on>1</always_on>
                 <visualize>true</visualize>
-                <topic>${namespace}/left</topic>
-                <!-- <ignition_frame_id>firefly_left_optical_frame</ignition_frame_id> -->
-                <camera name="firefly_left">
-                    <horizontal_fov>1.3962634</horizontal_fov>  <!-- 80 degrees -->
+                <topic>${namespace}/right</topic>
+                <camera name="firefly_right">
+                    <horizontal_fov>1.3962634</horizontal_fov>
                     <image>
                         <width>1440</width>
@@ -29,31 +58,5 @@
                 </camera>
             </sensor>
-        </gazebo>
-        <!-- Right Camera Sensor -->
-        <gazebo reference="firefly_right_optical_frame">
-            <sensor name="firefly_right_camera" type="camera">
-                <update_rate>30</update_rate>
-                <always_on>1</always_on>
-                <visualize>true</visualize>
-                <topic>${namespace}/right</topic>
-                <camera name="firefly_right">
-                    <horizontal_fov>1.3962634</horizontal_fov>  <!-- 80 degrees -->
-                    <image>
-                        <width>1440</width>
-                        <height>1080</height>
-                        <format>R8G8B8</format>
-                    </image>
-                    <clip>
-                        <near>0.01</near>
-                        <far>300</far>
-                    </clip>
-                    <noise>
-                        <type>gaussian</type>
-                        <mean>0.0</mean>
-                        <stddev>0.007</stddev>
-                    </noise>
-                </camera>
-            </sensor>
-        </gazebo>
+        </gazebo> -->
     </xacro:macro>
 </robot>

File: camera_ros2_wrappers/firefly-ros2-wrapper/firefly-ros2-wrapper-description/urdf/firefly_stereo_macro.urdf.xacro (robot description, xacro)
@@ -10,5 +10,5 @@
                 <origin xyz="0 0 0" rpy="0 0 0"/>
                 <geometry>
-                    <mesh filename="package://firefly-ros2-wrapper-description/meshes/firefly-stereo.dae" scale="1 1 1"/>
+                    <mesh filename="file://$(find firefly-ros2-wrapper-description)/meshes/firefly-stereo.dae" scale="1 1 1"/>
                 </geometry>
             </visual>
@@ -16,5 +16,5 @@
                 <origin xyz="0 0 0" rpy="0 0 0"/>
                 <geometry>
-                    <mesh filename="package://firefly-ros2-wrapper-description/meshes/firefly-stereo-collision.stl" scale="1 1 1"/>
+                    <mesh filename="file://$(find firefly-ros2-wrapper-description)/meshes/firefly-stereo-collision.stl" scale="1 1 1"/>
                 </geometry>
             </collision>
@@ -33,5 +33,5 @@
             <parent link="firefly_camera_link"/>
             <child link="firefly_right_optical_frame"/>
-            <origin xyz="0.02999871 0.07322070 0.00006055" rpy="${-pi/2} 0 0"/>
+            <origin xyz="0.02999871 0.07322070 0.00006055" rpy="0 0 ${pi/2}"/>
         </joint>
         <link name="firefly_left_optical_frame"/>
@@ -39,5 +39,5 @@
             <parent link="firefly_camera_link"/>
             <child link="firefly_left_optical_frame"/>
-            <origin xyz="-0.02999871 0.07322070 0.00006055" rpy="${-pi/2} 0 0"/>
+            <origin xyz="-0.02999871 0.07322070 0.00006055" rpy="0 0 ${pi/2}"/>
         </joint>
         <!-- Add Gazebo sensor plugins if in simulation -->

File: camera_ros2_wrappers/ximea-ros2-wrapper/ximea-ros2-wrapper-description/urdf/ximea_description.urdf.xacro (robot description, xacro)
@@ -2,5 +2,5 @@
 <robot name="ximea_camera" xmlns:xacro="http://ros.org/wiki/xacro">
     <!-- Include macro files -->
-    <xacro:include filename="$(find ximea_description)/urdf/ximea_macro.urdf.xacro" />
+    <xacro:include filename="$(find ximea-ros2-wrapper-description)/urdf/ximea_macro.urdf.xacro" />
     <xacro:ximea_camera/>
 </robot>

File: camera_ros2_wrappers/ximea-ros2-wrapper/ximea-ros2-wrapper-description/urdf/ximea_macro.urdf.xacro (robot description, xacro)
@@ -8,5 +8,5 @@
                 <origin xyz="0 0 0" rpy="0 0 0"/>
                 <geometry>
-                    <mesh filename="package://ximea_description/meshes/Ximea_Camera_EO_Lens.dae" scale="1 1 1"/>
+                    <mesh filename="file://$(find ximea-ros2-wrapper-description)/meshes/Ximea_Camera_EO_Lens.dae" scale="1 1 1"/>
                 </geometry>
             </visual>
@@ -14,5 +14,5 @@
                 <origin xyz="0 0 0" rpy="0 0 0"/>
                 <geometry>
-                    <mesh filename="package://ximea_description/meshes/Ximea_Camera_EO_Lens_Collision.stl" scale="1 1 1"/>
+                    <mesh filename="file://$(find ximea-ros2-wrapper-description)/meshes/Ximea_Camera_EO_Lens_Collision.stl" scale="1 1 1"/>
                 </geometry>
             </collision>

Commit message: Working to implement point cloud from simulated firefly images. At the moment, the stereo matching is providing less than ideal performance. I also broke the bringup for the firefly into a real and fake bringup for the moment. I also added my own stereo matching node because I was worried that the defualt one was not functioning properly.

File: camera_ros2_wrappers/firefly-ros2-wrapper/firefly-ros2-wrapper-description/urdf/firefly_stereo_gazebo.urdf.xacro (robot description, xacro)
@@ -3,15 +3,20 @@
     <!-- Gazebo (Ignition) sensor plugins for Firefly stereo camera -->
     <xacro:macro name="firefly_camera_gazebo" params="namespace:=firefly">
-        <!-- Sensors plugin must be loaded by world sdf for vision -->
+        <!-- Sensors plugin required for Ignition Gazebo camera simulation -->
+        <!-- <gazebo>
+            <plugin name="gz::sim::systems::Sensors" filename="libgz-sim-sensors-system.so">
+                <render_engine>ogre2</render_engine>
+            </plugin>
+        </gazebo> -->
         <!-- Left Camera Sensor -->
-        <gazebo reference="firefly_left_optical_frame">
+        <gazebo reference="firefly_left_camera_frame">
             <sensor name="firefly_left_camera" type="camera">
-                <update_rate>2</update_rate>
-                <always_on>1</always_on>
+                <update_rate>20</update_rate>
+                <always_on>true</always_on>
                 <visualize>true</visualize>
-                <topic>/camera</topic>
-                <gz_frame_id>firefly_left_optical_frame</gz_frame_id>
-                <!-- <optical_frame_id>firefly_left_optical_frame</optical_frame_id> -->
-                <!-- <camera_info_topic>/firefly_left/camera_info</camera_info_topic> -->
+                <topic>/firefly_left/image_raw</topic>
+                <ignition_frame_id>firefly_left_camera_optical_frame</ignition_frame_id>
+                <camera_info_topic>/firefly_left/camera_info</camera_info_topic>
+                <pose>0 0 0 0 0 0</pose>  <!-- Left camera at origin -->
                 <camera>
                     <horizontal_fov>1.3962634</horizontal_fov>  <!-- 80 degrees -->
@@ -23,6 +28,22 @@
                     <clip>
                         <near>0.1</near>
-                        <far>300</far>
+                        <far>10</far>
                     </clip>
+                    <!-- Left camera calibration matrix -->
+                    <!-- <intrinsics>
+                        <fx>858.0626964569092</fx>
+                        <fy>858.0626320838928</fy>
+                        <cx>720.0</cx>
+                        <cy>540.0</cy>
+                        <s>0.0</s>
+                    </intrinsics> -->
+                    <!-- <distortion>
+                        <k1>0.0</k1>
+                        <k2>0.0</k2>
+                        <k3>0.0</k3>
+                        <p1>0.0</p1>
+                        <p2>0.0</p2>
+                        <center>0.5 0.5</center>
+                    </distortion> -->
                     <!-- <noise>
                         <type>gaussian</type>
@@ -34,11 +55,14 @@
         </gazebo>
         <!-- Right Camera Sensor -->
-        <!-- <gazebo reference="firefly_right_optical_frame">
+        <gazebo reference="firefly_right_camera_frame">
             <sensor name="firefly_right_camera" type="camera">
-                <update_rate>30</update_rate>
-                <always_on>1</always_on>
+                <update_rate>20</update_rate>
+                <always_on>true</always_on>
                 <visualize>true</visualize>
-                <topic>${namespace}/right</topic>
-                <camera name="firefly_right">
+                <topic>/firefly_right/image_raw</topic>
+                <ignition_frame_id>firefly_right_camera_optical_frame</ignition_frame_id>
+                <camera_info_topic>/firefly_right/camera_info</camera_info_topic>
+                <pose>0 0 0 0 0 0</pose>  <!-- Create 6cm baseline for Gazebo stereo calibration -->
+                <camera>
                     <horizontal_fov>1.3962634</horizontal_fov>
                     <image>
@@ -49,14 +73,32 @@
                     <clip>
                         <near>0.01</near>
-                        <far>300</far>
+                        <far>10</far>
                     </clip>
-                    <noise>
+                    <!-- Right camera calibration matrix with stereo baseline -->
+                    <!-- <intrinsics>
+                        <fx>858.0626106262207</fx>
+                        <fy>858.0626964569092</fy>
+                        <cx>720.0</cx>
+                        <cy>540.0</cy>
+                        <s>0.0</s>
+                    </intrinsics> -->
+                    <!-- Stereo projection matrix with 6cm baseline -->
+                    <!-- -fx * baseline = -858.06 * 0.06 -->
+                    <!-- <projection>
+                        <p_fx>858.0626106262207</p_fx>
+                        <p_fy>858.0626964569092</p_fy>
+                        <p_cx>720.0</p_cx>
+                        <p_cy>540.0</p_cy>
+                        <tx>-51.48375</tx>
+                        <ty>0.0</ty>
+                    </projection> -->
+                    <!-- <noise>
                         <type>gaussian</type>
                         <mean>0.0</mean>
                         <stddev>0.007</stddev>
-                    </noise>
+                    </noise> -->
                 </camera>
             </sensor>
-        </gazebo> -->
+        </gazebo>
     </xacro:macro>
 </robot>

File: camera_ros2_wrappers/firefly-ros2-wrapper/firefly-ros2-wrapper-description/urdf/firefly_stereo_macro.urdf.xacro (robot description, xacro)
@@ -28,16 +28,29 @@
             </inertial>
         </link>
-        <!-- Optical frames for cameras -->
-        <link name="firefly_right_optical_frame"/>
-        <joint name="firefly_right_optical_joint" type="fixed">
+        <!-- Right camera and optical frames -->
+        <link name="firefly_right_camera_frame"/>
+        <joint name="firefly_right_camera_joint" type="fixed">
             <parent link="firefly_camera_link"/>
-            <child link="firefly_right_optical_frame"/>
+            <child link="firefly_right_camera_frame"/>
             <origin xyz="0.02999871 0.07322070 0.00006055" rpy="0 0 ${pi/2}"/>
         </joint>
-        <link name="firefly_left_optical_frame"/>
-        <joint name="firefly_left_optical_joint" type="fixed">
+        <link name="firefly_right_camera_optical_frame"/>
+        <joint name="firefly_right_camera_optical_joint" type="fixed">
+            <parent link="firefly_right_camera_frame"/>
+            <child link="firefly_right_camera_optical_frame"/>
+            <origin xyz="0 0 0" rpy="-${pi/2} 0 -${pi/2}"/>
+        </joint>
+        <!-- Left camera and optical frames -->
+        <link name="firefly_left_camera_frame"/>
+        <joint name="firefly_left_camera_joint" type="fixed">
             <parent link="firefly_camera_link"/>
-            <child link="firefly_left_optical_frame"/>
+            <child link="firefly_left_camera_frame"/>
             <origin xyz="-0.02999871 0.07322070 0.00006055" rpy="0 0 ${pi/2}"/>
+        </joint>
+        <link name="firefly_left_camera_optical_frame"/>
+        <joint name="firefly_left_camera_optical_joint" type="fixed">
+            <parent link="firefly_left_camera_frame"/>
+            <child link="firefly_left_camera_optical_frame"/>
+            <origin xyz="0 0 0" rpy="-${pi/2} 0 -${pi/2}"/>
         </joint>
         <!-- Add Gazebo sensor plugins if in simulation -->
