Commit message: Filled out the ximea bringup package. Added timer package which acts as a wrapper around the serial hw trigger module that Abhi built. This will now serve as the input for both the ximea and the firefly cameras because I modified the input cable to go to both cameras. I also recreated the gui module using some of the aspects of the previous one, but also adding a lot of configurability, faster displays, independent functionality across the different packages, and getting rid of the top-down director topic messaging system. We will sync afterwards as needed. This will work better for on-robot purposes as well.

File: multi_camera_rig_description/urdf/multi_camera_rig_description.urdf.xacro (robot description, xacro)
@@ -2,5 +2,5 @@
 <robot name="multi_camera_rig" xmlns:xacro="http://ros.org/wiki/xacro">
     <!-- Include macro files -->
-    <xacro:include filename="$(find multi_cam_rig_description)/urdf/multi_cam_rig_macro.urdf.xacro" />
+    <xacro:include filename="$(find multi_camera_rig_description)/urdf/multi_camera_rig_macro.urdf.xacro" />
     <xacro:multi_camera_rig/>
 </robot>

File: multi_camera_rig_description/urdf/multi_camera_rig_macro.urdf.xacro (robot description, xacro)
@@ -15,5 +15,5 @@
                 <origin xyz="0 0 0" rpy="0 0 0"/>
                 <geometry>
-                    <mesh filename="package://multi_cam_rig_description/meshes/Multi_Camera_Rig.dae" scale="1 1 1"/>
+                    <mesh filename="package://multi_camera_rig_description/meshes/Multi_Camera_Rig.dae" scale="1 1 1"/>
                 </geometry>
             </visual>
@@ -21,5 +21,5 @@
                 <origin xyz="0 0 0" rpy="0 0 0"/>
                 <geometry>
-                    <mesh filename="package://multi_cam_rig_description/meshes/Multi_Camera_Rig_Collision.stl" scale="1 1 1"/>
+                    <mesh filename="package://multi_camera_rig_description/meshes/Multi_Camera_Rig_Collision.stl" scale="1 1 1"/>
                 </geometry>
             </collision>
