Commit message: Renamed the camera wrapper folder, removed the ZED camera (since we aren't using it anyway), and moved the flir drivers to the external folder.

File: multi_camera_rig_description/urdf/multi_camera_rig_macro.urdf.xacro (robot description, xacro)
@@ -50,5 +50,5 @@
         </joint>
         <!-- ZED Camera -->
-        <xacro:include filename="$(find zed_wrapper)/urdf/zed_macro.urdf.xacro"/>
+        <!-- <xacro:include filename="$(find zed_wrapper)/urdf/zed_macro.urdf.xacro"/>
         <xacro:zed_camera name="zed2i"
                         model="zed2i"
@@ -61,5 +61,5 @@
             <child link="zed2i_camera_link"/>
             <origin xyz="0.0 0.05350000 -0.04838454" rpy="0 0 ${pi/2}"/>
-        </joint>
+        </joint> -->
     </xacro:macro>
 </robot>
