Commit message: Reduced camera mesh sizes.

File: multi_camera_rig_cameras/firefly-ros2-wrapper/firefly-ros2-wrapper-description/urdf/firefly_stereo_macro.urdf.xacro (robot description, xacro)
@@ -10,5 +10,5 @@
                 <origin xyz="0 0 0" rpy="0 0 0"/>
                 <geometry>
-                    <mesh filename="file://$(find firefly-ros2-wrapper-description)/meshes/firefly-stereo.dae" scale="1 1 1"/>
+                    <mesh filename="file://$(find firefly-ros2-wrapper-description)/meshes/FFS_Camera.obj" scale="1 1 1"/>
                 </geometry>
             </visual>

File: multi_camera_rig_cameras/ximea-ros2-wrapper/ximea-ros2-wrapper-description/urdf/ximea_macro.urdf.xacro (robot description, xacro)
@@ -8,5 +8,5 @@
                 <origin xyz="0 0 0" rpy="0 0 0"/>
                 <geometry>
-                    <mesh filename="file://$(find ximea-ros2-wrapper-description)/meshes/Ximea_Camera_EO_Lens.dae" scale="1 1 1"/>
+                    <mesh filename="file://$(find ximea-ros2-wrapper-description)/meshes/Ximea_Camera_EO_Lens.obj" scale="1 1 1"/>
                 </geometry>
             </visual>
