Commit message: Removed unneccessary source and launch files from the camera wrappers and updated thier cmakelists and package xml.

File: multi_camera_rig_cameras/firefly-ros2-wrapper/firefly-ros2-wrapper-description/urdf/firefly_stereo_gazebo.urdf.xacro (robot description, xacro)
@@ -2,5 +2,5 @@
 <robot xmlns:xacro="http://ros.org/wiki/xacro">
     <!-- Gazebo (Ignition) sensor plugins for Firefly stereo camera -->
-    <xacro:macro name="firefly_camera_gazebo" params="namespace:=firefly">
+    <xacro:macro name="firefly_camera_gazebo" params="namespace:=firefly frame_rate:=5">
         <!-- Sensors plugin required for Ignition Gazebo camera simulation -->
         <!-- We added this in the .sdf file for the world, but it can also be added here -->
@@ -8,5 +8,5 @@
         <gazebo reference="firefly_left_camera_frame">
             <sensor name="firefly_left_depth_camera" type="depth">
-                <update_rate>5</update_rate>
+                <update_rate>${frame_rate}</update_rate>
                 <visualize>false</visualize>
                 <topic>/firefly_left/sim/depth/image_raw</topic>
@@ -27,5 +27,5 @@
             </sensor>
             <sensor name="firefly_left_camera" type="camera">
-                <update_rate>5</update_rate>
+                <update_rate>${frame_rate}</update_rate>
                 <visualize>false</visualize>
                 <topic>/firefly_left/sim/image_raw</topic>
@@ -56,5 +56,5 @@
         <gazebo reference="firefly_right_camera_frame">
             <sensor name="firefly_right_depth_camera" type="depth">
-                <update_rate>5</update_rate>
+                <update_rate>${frame_rate}</update_rate>
                 <visualize>false</visualize>
                 <topic>/firefly_right/sim/depth/image_raw</topic>
@@ -75,5 +75,5 @@
             </sensor>
             <sensor name="firefly_right_camera" type="camera">
-                <update_rate>5</update_rate>
+                <update_rate>${frame_rate}</update_rate>
                 <visualize>false</visualize>
                 <topic>/firefly_right/sim/image_raw</topic>

File: multi_camera_rig_cameras/firefly-ros2-wrapper/firefly-ros2-wrapper-description/urdf/firefly_stereo_macro.urdf.xacro (robot description, xacro)
@@ -4,5 +4,5 @@
     <xacro:include filename="$(find firefly-ros2-wrapper-description)/urdf/firefly_stereo_gazebo.urdf.xacro"/>
     <!-- Macro Definition -->
-    <xacro:macro name="firefly_camera" params="use_gazebo:=true namespace:=firefly">
+    <xacro:macro name="firefly_camera" params="use_gazebo:=true namespace:=firefly frame_rate:=5">
         <!-- Link: camera body -->
         <link name="firefly_camera_link">
@@ -56,5 +56,5 @@
         <!-- Add Gazebo sensor plugins if in simulation -->
         <xacro:if value="${use_gazebo}">
-            <xacro:firefly_camera_gazebo namespace="${namespace}"/>
+            <xacro:firefly_camera_gazebo namespace="${namespace}" frame_rate="${frame_rate}"/>
         </xacro:if>
     </xacro:macro>

Commit message: Changed the default frame rate to lower the effort on the gazebo sim at the start.

File: multi_camera_rig_cameras/firefly-ros2-wrapper/firefly-ros2-wrapper-description/urdf/firefly_stereo_gazebo.urdf.xacro (robot description, xacro)
@@ -2,5 +2,5 @@
 <robot xmlns:xacro="http://ros.org/wiki/xacro">
     <!-- Gazebo (Ignition) sensor plugins for Firefly stereo camera -->
-    <xacro:macro name="firefly_camera_gazebo" params="namespace:=firefly frame_rate:=5">
+    <xacro:macro name="firefly_camera_gazebo" params="namespace:=firefly frame_rate:=1">
         <!-- Sensors plugin required for Ignition Gazebo camera simulation -->
         <!-- We added this in the .sdf file for the world, but it can also be added here -->

File: multi_camera_rig_cameras/firefly-ros2-wrapper/firefly-ros2-wrapper-description/urdf/firefly_stereo_macro.urdf.xacro (robot description, xacro)
@@ -4,5 +4,5 @@
     <xacro:include filename="$(find firefly-ros2-wrapper-description)/urdf/firefly_stereo_gazebo.urdf.xacro"/>
     <!-- Macro Definition -->
-    <xacro:macro name="firefly_camera" params="use_gazebo:=true namespace:=firefly frame_rate:=5">
+    <xacro:macro name="firefly_camera" params="use_gazebo:=true namespace:=firefly frame_rate:=1">
         <!-- Link: camera body -->
         <link name="firefly_camera_link">
